File: mechanical/transducer_board/transducer_board.sch (KiCad schematic (older format))
At the start: 63 parts, among them J1 Conn_02x17_Top_Bottom, J2 Conn_01x01, J3 Conn_01x01, U1 XL62783, U2 XL62083, U3 XL62783, U4 XL62083

Commit message: Completed transducer board layout
Parts:
- removed J1: Conn_02x17_Top_Bottom, Ultrasonic Emitters:PinHeader_2x17_P2.54mm_Vertical_SMD_Wide, symbol Connector_Generic:Conn_02x17_Top_Bottom
- added J1: Conn_02x17_Odd_Even, Ultrasonic Emitters:PinHeader_2x17_P2.54mm_Vertical_SMD_Wide, symbol Connector_Generic:Conn_02x17_Odd_Even
Other:
- moved on the sheet: C5, C6, C7, C8

Commit message: Transducers are driven with a bipolar waveform
Parts:
- added J4: Conn_01x01, Connector_Pin:Pin_D1.3mm_L11.0mm, symbol Connector_Generic:Conn_01x01
Connections:
- net labels added: VMID
- wire segments 169 -> 154
Other:
- moved on the sheet: J3
