File: electrical/fpga_board/fpga_board.kicad_pcb (KiCad board)
At the start: 4 copper layers, 92 x 92 mm, 52 parts, among them J1 Conn_02x17_Odd_Even, J10 Conn_01x01, J2 Conn_02x17_Odd_Even, J3 Conn_02x17_Odd_Even, J4 Conn_02x17_Odd_Even, J5 Conn_02x17_Odd_Even, J6 jtag, J7 Conn_02x03_Odd_Even, J8 Conn_02x12_Odd_Even, J9 Conn_01x01, U1 XC6SLX16-FTG256, U2 SiT1602, U3 MIC5504-3.3YM5, U4 MIC5504-1.2YM5

Commit message: Tweaks to PCBs
Routing:
- net /gnd: track 288.0 -> 278.2 mm
- net /T6+5: track 34.3 -> 28.5 mm
- net /T2+5: track 34.8 -> 29.2 mm
- net /T7+5: track 30.9 -> 25.4 mm
- net /T3+5: track 30.1 -> 24.7 mm
- net /T5+5: track 36.6 -> 31.8 mm
- net /T1+5: track 35.9 -> 31.2 mm
- net /T4+5: track 24.6 -> 19.9 mm
- net /vcc: track 369.9 -> 365.5 mm
- net /T5-5: track 24.1 -> 20.6 mm
- net /T1-5: track 22.5 -> 19.1 mm
- net /T8+5: track 25.2 -> 21.9 mm
- net /T6-5: track 22.8 -> 19.9 mm
- net /T2-5: track 21.3 -> 18.5 mm
- net /T6-3: track 98.2 -> 100.2 mm
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Other:
- board text added: "5V"
