File: electrical/transducer_board/transducer_board.sch (KiCad schematic (older format))
At the start: 64 parts, among them J1 Conn_02x17_Odd_Even, J2 Conn_01x01, J3 Conn_01x01, J4 Conn_01x01, U1 XL62783, U2 XL62083, U3 XL62783, U4 XL62083

Commit message: Tweaks to PCBs
Parts:
- C1, C2, C5, C6: footprint Capacitor_SMD:C_0805_2012Metric -> Capacitor_SMD:C_0603_1608Metric
- C3, C4, C7, C8: value .1uF -> 1uF; footprint Capacitor_SMD:C_0805_2012Metric -> Capacitor_SMD:C_0603_1608Metric
- R1, R10, R11, R12, R13, R14, R15, R16, R17, R18, R19, R2, R20, R21, R22, R23, R24, R25, R26, R27, R28, R29, R3, R30, R31, R32, R4, R5, R6, R7, R8, R9: value 620 -> 33
Changed lines of the file:
@@
 P 1150 2350
 F 0 "C3" H 1265 2396 50  0000 L CNN
-F 1 ".1uF" H 1265 2305 50  0000 L CNN
-F 2 "Capacitor_SMD:C_0805_2012Metric" H 1188 2200 50  0001 C CNN
+F 1 "1uF" H 1265 2305 50  0000 L CNN
+F 2 "Capacitor_SMD:C_0603_1608Metric" H 1188 2200 50  0001 C CNN
 F 3 "~" H 1150 2350 50  0001 C CNN
 	1    1150 2350
@@
 P 1150 4150
 F 0 "C4" H 1265 4196 50  0000 L CNN
-F 1 ".1uF" H 1265 4105 50  0000 L CNN
-F 2 "Capacitor_SMD:C_0805_2012Metric" H 1188 4000 50  0001 C CNN
+F 1 "1uF" H 1265 4105 50  0000 L CNN
+F 2 "Capacitor_SMD:C_0603_1608Metric" H 1188 4000 50  0001 C CNN
 F 3 "~" H 1150 4150 50  0001 C CNN
 	1    1150 4150
@@
 F 0 "C1" H 815 2396 50  0000 L CNN
 F 1 ".01uF" H 815 2305 50  0000 L CNN
-F 2 "Capacitor_SMD:C_0805_2012Metric" H 738 2200 50  0001 C CNN
+F 2 "Capacitor_SMD:C_0603_1608Metric" H 738 2200 50  0001 C CNN
 F 3 "~" H 700 2350 50  0001 C CNN
 	1    700  2350
@@
 F 0 "C2" H 815 4196 50  0000 L CNN
 F 1 ".01uF" H 815 4105 50  0000 L CNN
-F 2 "Capacitor_SMD:C_0805_2012Metric" H 738 4000 50  0001 C CNN
+F 2 "Capacitor_SMD:C_0603_1608Metric" H 738 4000 50  0001 C CNN
 F 3 "~" H 700 4150 50  0001 C CNN
 	1    700  4150
@@
 P 6850 1450
 F 0 "C7" H 6965 1496 50  0000 L CNN
-F 1 ".1uF" H 6965 1405 50  0000 L CNN
-F 2 "Capacitor_SMD:C_0805_2012Metric" H 6888 1300 50  0001 C CNN
+F 1 "1uF" H 6965 1405 50  0000 L CNN
+F 2 "Capacitor_SMD:C_0603_1608Metric" H 6888 1300 50  0001 C CNN
 F 3 "~" H 6850 1450 50  0001 C CNN
 	1    6850 1450
@@
 P 6900 3250
 F 0 "C8" H 7015 3296 50  0000 L CNN
-F 1 ".1uF" H 7015 3205 50  0000 L CNN
-F 2 "Capacitor_SMD:C_0805_2012Metric" H 6938 3100 50  0001 C CNN
+F 1 "1uF" H 7015 3205 50  0000 L CNN
+F 2 "Capacitor_SMD:C_0603_1608Metric" H 6938 3100 50  0001 C CNN
 F 3 "~" H 6900 3250 50  0001 C CNN
 	1    6900 3250
@@
 F 0 "C5" H 6515 1496 50  0000 L CNN
 F 1 ".01uF" H 6515 1405 50  0000 L CNN
-F 2 "Capacitor_SMD:C_0805_2012Metric" H 6438 1300 50  0001 C CNN
+F 2 "Capacitor_SMD:C_0603_1608Metric" H 6438 1300 50  0001 C CNN
 F 3 "~" H 6400 1450 50  0001 C CNN
 	1    6400 1450
@@
 F 0 "C6" H 6565 3296 50  0000 L CNN
 F 1 ".01uF" H 6565 3205 50  0000 L CNN
-F 2 "Capacitor_SMD:C_0805_2012Metric" H 6488 3100 50  0001 C CNN
+F 2 "Capacitor_SMD:C_0603_1608Metric" H 6488 3100 50  0001 C CNN
 F 3 "~" H 6450 3250 50  0001 C CNN
 	1    6450 3250
@@
 P 2250 2100
 F 0 "R12" V 2045 2100 50  0000 C CNN
-F 1 "620" V 2136 2100 50  0000 C CNN
+F 1 "33" V 2136 2100 50  0000 C CNN
 F 2 "Resistor_SMD:R_1206_3216Metric" V 2290 2090 50  0001 C CNN
 F 3 "~" H 2250 2100 50  0001 C CNN
@@
 P 2050 2000
 F 0 "R4" V 1845 2000 50  0000 C CNN
-F 1 "620" V 1936 2000 50  0000 C CNN
+F 1 "33" V 1936 2000 50  0000 C CNN
 F 2 "Resistor_SMD:R_1206_3216Metric" V 2090 1990 50  0001 C CNN
 F 3 "~" H 2050 2000 50  0001 C CNN
@@
 P 2250 1900
 F 0 "R11" V 2045 1900 50  0000 C CNN
-F 1 "620" V 2136 1900 50  0000 C CNN
+F 1 "33" V 2136 1900 50  0000 C CNN
 F 2 "Resistor_SMD:R_1206_3216Metric" V 2290 1890 50  0001 C CNN
 F 3 "~" H 2250 1900 50  0001 C CNN
@@
 P 2050 1800
 F 0 "R3" V 1845 1800 50  0000 C CNN
-F 1 "620" V 1936 1800 50  0000 C CNN
+F 1 "33" V 1936 1800 50  0000 C CNN
 F 2 "Resistor_SMD:R_1206_3216Metric" V 2090 1790 50  0001 C CNN
 F 3 "~" H 2050 1800 50  0001 C CNN
@@
 P 2250 1700
 F 0 "R10" V 2045 1700 50  0000 C CNN
-F 1 "620" V 2136 1700 50  0000 C CNN
+F 1 "33" V 2136 1700 50  0000 C CNN
 F 2 "Resistor_SMD:R_1206_3216Metric" V 2290 1690 50  0001 C CNN
 F 3 "~" H 2250 1700 50  0001 C CNN
@@
 P 2050 1600
 F 0 "R2" V 1845 1600 50  0000 C CNN
-F 1 "620" V 1936 1600 50  0000 C CNN
+F 1 "33" V 1936 1600 50  0000 C CNN
 F 2 "Resistor_SMD:R_1206_3216Metric" V 2090 1590 50  0001 C CNN
 F 3 "~" H 2050 1600 50  0001 C CNN
@@
 P 2250 1500
 F 0 "R9" V 2045 1500 50  0000 C CNN
-F 1 "620" V 2136 1500 50  0000 C CNN
+F 1 "33" V 2136 1500 50  0000 C CNN
 F 2 "Resistor_SMD:R_1206_3216Metric" V 2290 1490 50  0001 C CNN
 F 3 "~" H 2250 1500 50  0001 C CNN
@@
 P 2050 1400
 F 0 "R1" V 1845 1400 50  0000 C CNN
-F 1 "620" V 1936 1400 50  0000 C CNN
+F 1 "33" V 1936 1400 50  0000 C CNN
 F 2 "Resistor_SMD:R_1206_3216Metric" V 2090 1390 50  0001 C CNN
 F 3 "~" H 2050 1400 50  0001 C CNN
@@
 P 2050 3200
 F 0 "R5" V 1845 3200 50  0000 C CNN
-F 1 "620" V 1936 3200 50  0000 C CNN
+F 1 "33" V 1936 3200 50  0000 C CNN
 F 2 "Resistor_SMD:R_1206_3216Metric" V 2090 3190 50  0001 C CNN
 F 3 "~" H 2050 3200 50  0001 C CNN
@@
 P 2250 3300
 F 0 "R13" V 2045 3300 50  0000 C CNN
-F 1 "620" V 2136 3300 50  0000 C CNN
+F 1 "33" V 2136 3300 50  0000 C CNN
 F 2 "Resistor_SMD:R_1206_3216Metric" V 2290 3290 50  0001 C CNN
 F 3 "~" H 2250 3300 50  0001 C CNN
@@
 P 2050 3400
 F 0 "R6" V 1845 3400 50  0000 C CNN
-F 1 "620" V 1936 3400 50  0000 C CNN
+F 1 "33" V 1936 3400 50  0000 C CNN
 F 2 "Resistor_SMD:R_1206_3216Metric" V 2090 3390 50  0001 C CNN
 F 3 "~" H 2050 3400 50  0001 C CNN
@@
 P 2050 3600
 F 0 "R7" V 1845 3600 50  0000 C CNN
-F 1 "620" V 1936 3600 50  0000 C CNN
+F 1 "33" V 1936 3600 50  0000 C CNN
 F 2 "Resistor_SMD:R_1206_3216Metric" V 2090 3590 50  0001 C CNN
 F 3 "~" H 2050 3600 50  0001 C CNN
@@
 P 2050 3800
 F 0 "R8" V 1845 3800 50  0000 C CNN
-F 1 "620" V 1936 3800 50  0000 C CNN
+F 1 "33" V 1936 3800 50  0000 C CNN
 F 2 "Resistor_SMD:R_1206_3216Metric" V 2090 3790 50  0001 C CNN
 F 3 "~" H 2050 3800 50  0001 C CNN
@@
 P 2250 3500
 F 0 "R14" V 2045 3500 50  0000 C CNN
-F 1 "620" V 2136 3500 50  0000 C CNN
+F 1 "33" V 2136 3500 50  0000 C CNN
 F 2 "Resistor_SMD:R_1206_3216Metric" V 2290 3490 50  0001 C CNN
 F 3 "~" H 2250 3500 50  0001 C CNN
@@
 P 2250 3700
 F 0 "R15" V 2045 3700 50  0000 C CNN
-F 1 "620" V 2136 3700 50  0000 C CNN
+F 1 "33" V 2136 3700 50  0000 C CNN
 F 2 "Resistor_SMD:R_1206_3216Metric" V 2290 3690 50  0001 C CNN
 F 3 "~" H 2250 3700 50  0001 C CNN
@@
 P 2250 3900
 F 0 "R16" V 2045 3900 50  0000 C CNN
-F 1 "620" V 2136 3900 50  0000 C CNN
+F 1 "33" V 2136 3900 50  0000 C CNN
 F 2 "Resistor_SMD:R_1206_3216Metric" V 2290 3890 50  0001 C CNN
 F 3 "~" H 2250 3900 50  0001 C CNN
@@
 P 8350 2100
 F 0 "R28" V 8145 2100 50  0000 C CNN
-F 1 "620" V 8236 2100 50  0000 C CNN
+F 1 "33" V 8236 2100 50  0000 C CNN
 F 2 "Resistor_SMD:R_1206_3216Metric" V 8390 2090 50  0001 C CNN
 F 3 "~" H 8350 2100 50  0001 C CNN
@@
 P 8150 2000
 F 0 "R20" V 7945 2000 50  0000 C CNN
-F 1 "620" V 8036 2000 50  0000 C CNN
+F 1 "33" V 8036 2000 50  0000 C CNN
 F 2 "Resistor_SMD:R_1206_3216Metric" V 8190 1990 50  0001 C CNN
 F 3 "~" H 8150 2000 50  0001 C CNN
@@
 P 8350 1900
 F 0 "R27" V 8145 1900 50  0000 C CNN
-F 1 "620" V 8236 1900 50  0000 C CNN
+F 1 "33" V 8236 1900 50  0000 C CNN
 F 2 "Resistor_SMD:R_1206_3216Metric" V 8390 1890 50  0001 C CNN
 F 3 "~" H 8350 1900 50  0001 C CNN
@@
 P 8150 1800
 F 0 "R19" V 7945 1800 50  0000 C CNN
-F 1 "620" V 8036 1800 50  0000 C CNN
+F 1 "33" V 8036 1800 50  0000 C CNN
 F 2 "Resistor_SMD:R_1206_3216Metric" V 8190 1790 50  0001 C CNN
 F 3 "~" H 8150 1800 50  0001 C CNN
@@
 P 8350 1700
 F 0 "R26" V 8145 1700 50  0000 C CNN
-F 1 "620" V 8236 1700 50  0000 C CNN
+F 1 "33" V 8236 1700 50  0000 C CNN
 F 2 "Resistor_SMD:R_1206_3216Metric" V 8390 1690 50  0001 C CNN
 F 3 "~" H 8350 1700 50  0001 C CNN
@@
 P 8150 1600
 F 0 "R18" V 7945 1600 50  0000 C CNN
-F 1 "620" V 8036 1600 50  0000 C CNN
+F 1 "33" V 8036 1600 50  0000 C CNN
 F 2 "Resistor_SMD:R_1206_3216Metric" V 8190 1590 50  0001 C CNN
 F 3 "~" H 8150 1600 50  0001 C CNN
@@
 P 8350 1500
 F 0 "R25" V 8145 1500 50  0000 C CNN
-F 1 "620" V 8236 1500 50  0000 C CNN
+F 1 "33" V 8236 1500 50  0000 C CNN
 F 2 "Resistor_SMD:R_1206_3216Metric" V 8390 1490 50  0001 C CNN
 F 3 "~" H 8350 1500 50  0001 C CNN
@@
 P 8150 1400
 F 0 "R17" V 7945 1400 50  0000 C CNN
-F 1 "620" V 8036 1400 50  0000 C CNN
+F 1 "33" V 8036 1400 50  0000 C CNN
 F 2 "Resistor_SMD:R_1206_3216Metric" V 8190 1390 50  0001 C CNN
 F 3 "~" H 8150 1400 50  0001 C CNN
@@
 P 8150 3200
 F 0 "R21" V 7945 3200 50  0000 C CNN
-F 1 "620" V 8036 3200 50  0000 C CNN
+F 1 "33" V 8036 3200 50  0000 C CNN
 F 2 "Resistor_SMD:R_1206_3216Metric" V 8190 3190 50  0001 C CNN
 F 3 "~" H 8150 3200 50  0001 C CNN
@@
 P 8350 3300
 F 0 "R29" V 8145 3300 50  0000 C CNN
-F 1 "620" V 8236 3300 50  0000 C CNN
+F 1 "33" V 8236 3300 50  0000 C CNN
 F 2 "Resistor_SMD:R_1206_3216Metric" V 8390 3290 50  0001 C CNN
 F 3 "~" H 8350 3300 50  0001 C CNN
@@
 P 8150 3400
 F 0 "R22" V 7945 3400 50  0000 C CNN
-F 1 "620" V 8036 3400 50  0000 C CNN
+F 1 "33" V 8036 3400 50  0000 C CNN
 F 2 "Resistor_SMD:R_1206_3216Metric" V 8190 3390 50  0001 C CNN
 F 3 "~" H 8150 3400 50  0001 C CNN
@@
 P 8150 3600
 F 0 "R23" V 7945 3600 50  0000 C CNN
-F 1 "620" V 8036 3600 50  0000 C CNN
+F 1 "33" V 8036 3600 50  0000 C CNN
 F 2 "Resistor_SMD:R_1206_3216Metric" V 8190 3590 50  0001 C CNN
 F 3 "~" H 8150 3600 50  0001 C CNN
@@
 P 8150 3800
 F 0 "R24" V 7945 3800 50  0000 C CNN
-F 1 "620" V 8036 3800 50  0000 C CNN
+F 1 "33" V 8036 3800 50  0000 C CNN
 F 2 "Resistor_SMD:R_1206_3216Metric" V 8190 3790 50  0001 C CNN
 F 3 "~" H 8150 3800 50  0001 C CNN
@@
 P 8350 3500
 F 0 "R30" V 8145 3500 50  0000 C CNN
-F 1 "620" V 8236 3500 50  0000 C CNN
+F 1 "33" V 8236 3500 50  0000 C CNN
 F 2 "Resistor_SMD:R_1206_3216Metric" V 8390 3490 50  0001 C CNN
 F 3 "~" H 8350 3500 50  0001 C CNN
@@
 P 8350 3700
 F 0 "R31" V 8145 3700 50  0000 C CNN
-F 1 "620" V 8236 3700 50  0000 C CNN
+F 1 "33" V 8236 3700 50  0000 C CNN
 F 2 "Resistor_SMD:R_1206_3216Metric" V 8390 3690 50  0001 C CNN
 F 3 "~" H 8350 3700 50  0001 C CNN
@@
 P 8350 3900
 F 0 "R32" V 8145 3900 50  0000 C CNN
-F 1 "620" V 8236 3900 50  0000 C CNN
+F 1 "33" V 8236 3900 50  0000 C CNN
 F 2 "Resistor_SMD:R_1206_3216Metric" V 8390 3890 50  0001 C CNN
 F 3 "~" H 8350 3900 50  0001 C CNN

Commit message: Switched to FPGA on transducer board
Parts:
- removed J1: Conn_02x17_Odd_Even, Ultrasonic Emitters:PinHeader_2x17_P2.54mm_Vertical_SMD_Wide, symbol Connector_Generic:Conn_02x17_Odd_Even
- added C10, C12, C13, C14, C20, C24, C25: 100nF, Capacitor_SMD:C_0603_1608Metric, symbol Device:C
- added C11, C23, C9: 10uF, Capacitor_SMD:C_0805_2012Metric, symbol Device:C
- added C15, C16, C17, C18, C19: 1uF, Capacitor_SMD:C_0603_1608Metric, symbol Device:C
- added C21, C22: 10nF, Capacitor_SMD:C_0402_1005Metric, symbol Device:C
- added J1: Conn_01x04_MountingPin, Connector_JST:JST_SH_BM04B-SRSS-TB_1x04-1MP_P1.00mm_Vertical, symbol Connector_Generic_MountingPin:Conn_01x04_MountingPin
- added J14, J6: Conn_01x01, Connector_Pin:Pin_D1.0mm_L10.0mm, symbol Connector_Generic:Conn_01x01
- added J9: Conn_01x01, Connector_Pin:Pin_D1.3mm_L11.0mm, symbol Connector_Generic:Conn_01x01
- added R33: 10k, Resistor_SMD:R_0603_1608Metric, symbol Device:R_US
- added R34, R36: 4.7k, Resistor_SMD:R_0402_1005Metric, symbol Device:R_US
- added R35: 100, Resistor_SMD:R_0402_1005Metric, symbol Device:R_US
- added U5: ICE5LP1K-SG48, Package_DFN_QFN:QFN-48-1EP_7x7mm_P0.5mm_EP5.6x5.6mm, symbol FPGA_Lattice:ICE5LP1K-SG48
- added U6: MIC5504-1.2YM5, Package_TO_SOT_SMD:SOT-23-5, symbol Regulator_Linear:MIC5504-1.2YM5
- added U7: MIC5504-3.3YM5, Package_TO_SOT_SMD:SOT-23-5, symbol Regulator_Linear:MIC5504-3.3YM5
- added U8: 74LVC3G34, Package_SO:VSSOP-8_2.3x2mm_P0.5mm, symbol Ultrasonic~Library:74LVC3G34
- added X1: S3D10.000000B20F30T, Oscillator:Oscillator_SMD_Abracon_ASE-4Pin_3.2x2.5mm, symbol Oscillator:ASE-xxxMHz
- C1, C2, C5, C6: value .01uF -> 100nF
Connections:
- net labels added: CDONE, CLK, CRESET, GPIO_1, SCK, SPI_SI, SPI_SS, SYNC, T12+_OD, T16+_OD, V_1.2, V_3.3, V_5
- wire segments 154 -> 239
- no-connect marks 2 -> 3
Other:
- moved on the sheet: J2, J3, J4

Commit message: Switched to MachXO3 FPGA
Also switched to Kicad 6
Parts:
- removed C21: 10nF, Capacitor_SMD:C_0402_1005Metric, symbol Device:C
- removed C23: 10uF, Capacitor_SMD:C_0805_2012Metric, symbol Device:C
- removed C24: 100nF, Capacitor_SMD:C_0603_1608Metric, symbol Device:C
- removed J14: Conn_01x01, Connector_Pin:Pin_D1.0mm_L10.0mm, symbol Connector_Generic:Conn_01x01
- removed R35: 100, Resistor_SMD:R_0402_1005Metric, symbol Device:R_US
- removed U5: ICE5LP1K-SG48, Package_DFN_QFN:QFN-48-1EP_7x7mm_P0.5mm_EP5.6x5.6mm, symbol FPGA_Lattice:ICE5LP1K-SG48
- added U5: LCMXO3L-2100E-5UWG49, Ultrasonic Emitters:WLCSP-49-Lattice, symbol Ultrasonic~Library:LCMXO3L-2100E-5UWG49
Connections:
- net labels added: JTAGENB
- net labels removed: CDONE, CRESET
- wire segments 239 -> 243
- no-connect marks 3 -> 1
Other:
- note added: "Buffer exists b/c driver chips aren't CMOS - they draw a little current, so a pullup resistor might change their behavior"
- moved on the sheet: C10, C12, C14, C19, C20, C22
