File: electrical/transducer_board/transducer_board.kicad_pcb (KiCad board)
At the start: 4 copper layers, 66.6 x 66.6 mm, 90 parts, among them J1 Conn_01x04_MountingPin, J2 Conn_01x01, J3 Conn_01x01, J4 Conn_01x01, J6 Conn_01x01, J9 Conn_01x01, U1 XL62783, U2 XL62083, U3 XL62783, U4 XL62083, U5 LCMXO3L-2100E-5UWG49, U6 ME6211C12M5G-N, U7 PJ9193M33SE, U8 74LVC3G34, X1 X1G004171001600

Commit message: Add a few components
Parts:
- added C23: 100nF, Capacitor_SMD:C_0603_1608Metric, F.Cu at (143.5, 134.0)
- added C24: 100nF, Capacitor_SMD:C_0603_1608Metric, F.Cu at (142.2, 152.7)
- added C26: 100nF, Capacitor_SMD:C_0603_1608Metric, F.Cu at (122.2, 154.7)
- added C27: 100nF, Capacitor_SMD:C_0603_1608Metric, F.Cu at (128.3, 142.7)
- added C28: 100nF, Capacitor_SMD:C_0603_1608Metric, F.Cu at (118.1, 133.7)
- added C29: 100nF, Capacitor_SMD:C_0603_1608Metric, F.Cu at (101.9, 117.2)
- added D1: D, Diode_SMD:D_SOD-123, F.Cu at (109.2, 105.3)
- added D2: D, Diode_SMD:D_SOD-123, F.Cu at (98.5, 107.2)
- R1, R10, R11, R12, R13, R14, R15, R16, R17, R18, R19, R2, R20, R21, R22, R23, R24, R25, R26, R27, R28, R29, R3, R30, R31, R32, R4, R5, R6, R7, R8, R9: value 50 -> 47
- moved C4 8.51 mm to (133.8, 152.5)
- moved C2 8.51 mm to (133.7, 150.2)
- moved C6 8.33 mm to (108.5, 135.2)
- moved C8 8.33 mm to (108.5, 133.0)
- moved R12 5.15 mm to (131.6, 155.6)
- moved R16 3.65 mm to (137.8, 155.6)
- moved C18 1.97 mm to (109.0, 102.0)
Connections:
- C1 pad 2: GND -> /VMID
- C15 pad 1: /V_3.3 -> /V_3.3_D
- C16 pad 1: /V_5 -> /V_5_D
- C2 pad 1: VCC -> /VMID
- C3 pad 2: GND -> /VMID
- C4 pad 1: VCC -> /VMID
- C5 pad 2: GND -> /VMID
- C6 pad 1: VCC -> /VMID
- C7 pad 2: GND -> /VMID
- C8 pad 1: VCC -> /VMID
- U6 pad 1: /V_3.3 -> /V_3.3_D
- U6 pad 3: /V_3.3 -> /V_3.3_D
- U7 pad 1: /V_5 -> /V_5_D
- U7 pad 3: /V_5 -> /V_5_D
Routing:
- net /VMID: track 321.9 -> 20.7 mm, vias 2 -> 8
- net /V_3.3_D: track 0.00 -> 11.6 mm
- net /V_5_D: track 0.00 -> 9.67 mm
- net Net-(LS6-Pad1): track 43.3 -> 33.9 mm, vias 3 -> 2
- net /V_3.3: track 115.0 -> 106.4 mm
- net /V_5: track 10.9 -> 4.15 mm
- net Net-(R12-Pad2): track 27.4 -> 33.7 mm
- net /T10-: track 45.9 -> 39.7 mm
- net Net-(R17-Pad2): track 70.5 -> 64.6 mm
- net Net-(LS8-Pad1): track 7.56 -> 12.6 mm
- net Net-(R32-Pad2): track 34.8 -> 39.3 mm
- net Net-(R5-Pad2): track 47.3 -> 51.7 mm
- net Net-(R24-Pad2): track 27.4 -> 31.3 mm
- net Net-(R21-Pad2): track 37.8 -> 40.3 mm
- net Net-(R13-Pad2): track 59.1 -> 61.5 mm
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Other:
- board text added: "SPARC"
